File: Hardware/stm32F4V2.kicad_sch (KiCad schematic)
At the start: 38 parts, among them J1 USB_C_Receptacle_USB2.0_16P, J2 Conn_01x04, J5 Conn_01x18, J6 Conn_01x18, SW1 Push, SW3 Push, U1 STM32F411CCU6, U2 AZ1117-3.3, U4 2SC6, Y2 8MHz

Commit message: Finalized Layout for V.1
Parts:
- C12: footprint Capacitor_SMD:C_0402_1005Metric -> Capacitor_SMD:C_0603_1608Metric; Distributor Link https://www.digikey.com/en/products/detail/nextgen-componen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 -> https://www.digikey.com/en/products/detail/samsung-electro-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; Manufacturer Aillen -> Samsung Electro-Mechanics; Manufacturer Part Number 0402W106M6R3HI -> CL10A106MQ8NNNC
- C14, C15: value 10pF -> 10p
- C6: Distributor Link https://www.digikey.com/en/products/detail/nextgen-componen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 -> https://www.digikey.com/en/products/detail/murata-electroni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; Manufacturer Aillen -> Murata Electronics; Manufacturer Part Number 0402W105K100HI -> GRM155R70J105KA12D
Other:
- note added: "LDO"
- note removed: "Power Regulator"
- moved on the sheet: J2, TP1
Changed lines of the file:
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@@
 	(wire
 		(pts
-			(xy 175.26 149.86) (xy 186.69 149.86)
+			(xy 184.15 142.24) (xy 195.58 142.24)
 		)
 		(stroke
@@
 	(wire
 		(pts
-			(xy 128.27 187.96) (xy 128.27 190.5)
+			(xy 255.27 57.15) (xy 255.27 59.69)
 		)
 		(stroke
@@
 	(polyline
 		(pts
-			(xy 173.99 133.35) (xy 182.88 133.35)
+			(xy 182.88 125.73) (xy 191.77 125.73)
 		)
 		(stroke
@@
 	(wire
 		(pts
-			(xy 175.26 144.78) (xy 177.8 144.78)
+			(xy 184.15 137.16) (xy 186.69 137.16)
 		)
 		(stroke
@@
 	(wire
 		(pts
-			(xy 177.8 152.4) (xy 177.8 158.75)
+			(xy 186.69 144.78) (xy 186.69 151.13)
 		)
 		(stroke
@@
 	(wire
 		(pts
-			(xy 175.26 152.4) (xy 177.8 152.4)
+			(xy 184.15 144.78) (xy 186.69 144.78)
 		)
 		(stroke
@@
 	(polyline
 		(pts
-			(xy 182.88 162.56) (xy 163.83 162.56)
+			(xy 191.77 154.94) (xy 172.72 154.94)
 		)
 		(stroke
@@
 	(wire
 		(pts
-			(xy 175.26 147.32) (xy 186.69 147.32)
+			(xy 184.15 139.7) (xy 195.58 139.7)
 		)
 		(stroke
@@
 	(wire
 		(pts
-			(xy 177.8 139.7) (xy 177.8 144.78)
+			(xy 186.69 132.08) (xy 186.69 137.16)
 		)
 		(stroke
@@
 	(polyline
 		(pts
-			(xy 182.88 133.35) (xy 191.77 133.35)
+			(xy 191.77 125.73) (xy 200.66 125.73)
 		)
 		(stroke
@@
 	(polyline
 		(pts
-			(xy 163.83 162.56) (xy 163.83 133.35)
+			(xy 172.72 154.94) (xy 172.72 125.73)
 		)
 		(stroke
@@
 	(polyline
 		(pts
-			(xy 163.83 133.35) (xy 175.26 133.35)
+			(xy 172.72 125.73) (xy 184.15 125.73)
 		)
 		(stroke
@@
 	(polyline
 		(pts
-			(xy 191.77 162.56) (xy 181.61 162.56)
+			(xy 200.66 154.94) (xy 190.5 154.94)
 		)
 		(stroke
@@
 	(polyline
 		(pts
-			(xy 191.77 133.35) (xy 191.77 162.56)
+			(xy 200.66 125.73) (xy 200.66 154.94)
 		)
 		(stroke
@@
 		)
 	)
-	(text "Power Regulator\n"
+	(text "LDO"
 		(exclude_from_sim no)
 		(at 33.02 91.948 0)
@@
 	(text "SWD Header\n"
 		(exclude_from_sim no)
-		(at 169.926 134.874 0)
+		(at 178.816 127.254 0)
 		(effects
 			(font
@@
 	)
 	(label "SWD_DIO"
-		(at 179.07 147.32 0)
+		(at 187.96 139.7 0)
 		(fields_autoplaced yes)
 		(effects
@@
 	)
 	(label "SWD_CLK"
-		(at 179.07 149.86 0)
+		(at 187.96 142.24 0)
 		(fields_autoplaced yes)
 		(effects
@@
 			)
 		)
-		(property "Distributor Link" "https://www.digikey.com/en/products/detail/nextgen-components/0402W105K100HI/14632388?s=N4IgjCBcpgLFoDGUBmBDANgZwKYBoQB7KAbRAHZYBWMKkAXQIAcAXKEAZRYCcBLAOwDmIAL4EATAAZYATgQhkkdNnxFS4AAQBWgGINmbSCACq-XiwDyKALI40WAK7ccoggFp40Baky4CxSDIZAGY4CHoRMRAANnleABN2NzBJcRADdnSQFgBPJhcjeKxkSKA"
+		(property "Distributor Link" "https://www.digikey.com/en/products/detail/murata-electronics/GRM155R70J105KA12D/5027109"
 			(at 160.02 44.45 0)
 			(effects
@@
 			)
 		)
-		(property "Manufacturer" "Aillen"
+		(property "Manufacturer" "Murata Electronics"
 			(at 160.02 44.45 0)
 			(effects
@@
 			)
 		)
-		(property "Manufacturer Part Number" "0402W105K100HI"
+		(property "Manufacturer Part Number" "GRM155R70J105KA12D"
 			(at 160.02 44.45 0)
 			(effects
@@
 	(symbol
 		(lib_id "power:+3.3V")
-		(at 177.8 139.7 0)
+		(at 186.69 132.08 0)
 		(unit 1)
 		(exclude_from_sim no)
@@
 		(dnp no)
 		(property "Reference" "#PWR022"
-			(at 177.8 143.51 0)
+			(at 186.69 135.89 0)
 			(effects
 				(font
@@
 		)
 		(property "Value" "+3.3V"
-			(at 177.8 136.144 0)
+			(at 186.69 128.524 0)
 			(effects
 				(font
@@
 		)
 		(property "Footprint" ""
-			(at 177.8 139.7 0)
+			(at 186.69 132.08 0)
 			(effects
 				(font
@@
 		)
 		(property "Datasheet" ""
-			(at 177.8 139.7 0)
+			(at 186.69 132.08 0)
 			(effects
 				(font
@@
 		)
 		(property "Description" "Power symbol creates a global label with name \"+3.3V\""
-			(at 177.8 139.7 0)
+			(at 186.69 132.08 0)
 			(effects
 				(font
@@
 	(symbol
 		(lib_id "power:GND")
-		(at 177.8 158.75 0)
+		(at 186.69 151.13 0)
 		(unit 1)
 		(exclude_from_sim no)
@@
 		(fields_autoplaced yes)
 		(property "Reference" "#PWR021"
-			(at 177.8 165.1 0)
+			(at 186.69 157.48 0)
 			(effects
 				(font
@@
 		)
 		(property "Value" "GND"
-			(at 177.8 163.83 0)
+			(at 186.69 156.21 0)
 			(effects
 				(font
@@
 		)
 		(property "Footprint" ""
-			(at 177.8 158.75 0)
+			(at 186.69 151.13 0)
 			(effects
 				(font
@@
 		)
 		(property "Datasheet" ""
-			(at 177.8 158.75 0)
+			(at 186.69 151.13 0)
 			(effects
 				(font
@@
 		)
 		(property "Description" "Power symbol creates a global label with name \"GND\" , ground"
-			(at 177.8 158.75 0)
+			(at 186.69 151.13 0)
 			(effects
 				(font
@@
 			)
 		)
-		(property "Value" "10pF"
+		(property "Value" "10p"
 			(at 22.86 41.9099 0)
 			(effects
@@
 			)
 		)
-		(property "Footprint" "Capacitor_SMD:C_0402_1005Metric"
+		(property "Footprint" "Capacitor_SMD:C_0603_1608Metric"
 			(at 20.0152 111.76 0)
 			(effects
@@
 			)
 		)
-		(property "Distributor Link" "https://www.digikey.com/en/products/detail/nextgen-components/0402W106M6R3HI/18677011?s=N4IgjCBcoEwAwBYCcVQGMoDMCGAbAzgKYA0IA9lANrhwAEArQGIgC6pADgC5QgCqAdgEtOAeUwBZQtnwBXAE6EQAX1IBaBKhAZIOAiXJUQSAMxgEEFkpUgAbJsEATHqrBwYIDt0ggPITgE92RW8HfAwrIA"
+		(property "Distributor Link" "https://www.digikey.com/en/products/detail/samsung-electro-mechanics/CL10A106MQ8NNNC/3886777"
 			(at 19.05 107.95 0)
 			(effects
@@
 			)
 		)
-		(property "Manufacturer" "Aillen"
+		(property "Manufacturer" "Samsung Electro-Mechanics"
 			(at 19.05 107.95 0)
 			(effects
@@
 			)
 		)
-		(property "Manufacturer Part Number" "0402W106M6R3HI"
+		(property "Manufacturer Part Number" "CL10A106MQ8NNNC"
 			(at 19.05 107.95 0)
 			(effects
@@
 			)
 		)
-		(property "Value" "10pF"
+		(property "Value" "10p"
 			(at 42.164 41.148 0)
 			(effects
@@
 	(symbol
 		(lib_id "power:GND")
-		(at 128.27 190.5 0)
+		(at 255.27 59.69 0)
 		(unit 1)
 		(exclude_from_sim no)
@@
 		(fields_autoplaced yes)
 		(property "Reference" "#PWR027"
-			(at 128.27 196.85 0)
+			(at 255.27 66.04 0)
 			(effects
 				(font
@@
 		)
 		(property "Value" "GND"
-			(at 128.27 195.58 0)
+			(at 255.27 64.77 0)
 			(effects
 				(font
@@
 		)
 		(property "Footprint" ""
-			(at 128.27 190.5 0)
+			(at 255.27 59.69 0)
 			(effects
 				(font
@@
 		)
 		(property "Datasheet" ""
-			(at 128.27 190.5 0)
+			(at 255.27 59.69 0)
 			(effects
 				(font
@@
 		)
 		(property "Description" "Power symbol creates a global label with name \"GND\" , ground"
-			(at 128.27 190.5 0)
+			(at 255.27 59.69 0)
 			(effects
 				(font
@@
 	(symbol
 		(lib_id "Connector_Generic:Conn_01x04")
-		(at 170.18 147.32 0)
+		(at 179.07 139.7 0)
 		(mirror y)
 		(unit 1)
@@
 		(dnp no)
 		(property "Reference" "J2"
-			(at 170.18 142.24 0)
+			(at 179.07 134.62 0)
 			(effects
 				(font
@@
 		)
 		(property "Value" "Conn_01x04"
-			(at 171.704 155.194 0)
+			(at 180.594 147.574 0)
 			(effects
 				(font
@@
 		)
 		(property "Footprint" "Connector_PinHeader_2.54mm:PinHeader_1x04_P2.54mm_Vertical"
-			(at 170.18 147.32 0)
+			(at 179.07 139.7 0)
 			(effects
 				(font
@@
 		)
 		(property "Datasheet" "~"
-			(at 170.18 147.32 0)
+			(at 179.07 139.7 0)
 			(effects
 				(font
@@
 		)
 		(property "Description" "Generic connector, single row, 01x04, script generated (kicad-library-utils/schlib/autogen/connector/)"
-			(at 170.18 147.32 0)
+			(at 179.07 139.7 0)
 			(effects
 				(font
@@
 		)
 		(property "Distributor Link" "https://www.digikey.com/en/products/detail/w%C3%BCrth-elektronik/61300411121/4846827"
-			(at 170.18 147.32 0)
+			(at 179.07 139.7 0)
 			(effects
 				(font
@@
 		)
 		(property "Manufacturer" "Würth Elektronik"
-			(at 170.18 147.32 0)
+			(at 179.07 139.7 0)
 			(effects
 				(font
@@
 		)
 		(property "Manufacturer Part Number" "61300411121"
-			(at 170.18 147.32 0)
+			(at 179.07 139.7 0)
 			(effects
 				(font
@@
 	(symbol
 		(lib_id "Connector:TestPoint")
-		(at 128.27 187.96 0)
+		(at 255.27 57.15 0)
 		(unit 1)
 		(exclude_from_sim no)
@@
 		(fields_autoplaced yes)
 		(property "Reference" "TP1"
-			(at 130.81 183.3879 0)
+			(at 257.81 52.5779 0)
 			(effects
 				(font
@@
 		)
 		(property "Value" "TestPoint"
-			(at 130.81 185.9279 0)
+			(at 257.81 55.1179 0)
 			(effects
 				(font
@@
 		)
 		(property "Footprint" "TestPoint:TestPoint_Pad_2.0x2.0mm"
-			(at 133.35 187.96 0)
+			(at 260.35 57.15 0)
 			(effects
 				(font
@@
 		)
 		(property "Datasheet" "~"
-			(at 133.35 187.96 0)
+			(at 260.35 57.15 0)
 			(effects
 				(font
@@
 		)
 		(property "Description" "test point"
-			(at 128.27 187.96 0)
+			(at 255.27 57.15 0)
 			(effects
 				(font
